Commit message: Solved the URDF issues

File: bimur/bimur_description/urdf/inc/ur5_macro.xacro (robot description, xacro)
@@ -20,5 +20,5 @@
   <xacro:include filename="$(find ur_description)/urdf/inc/ur_common.xacro" />
   <xacro:macro name="ur5_robot" params="
-    prefix
+    prefix:=''
     joint_limits_parameters_file:='$(find ur_description)/config/ur5/joint_limits.yaml'
     kinematics_parameters_file:='$(find ur_description)/config/ur5/default_kinematics.yaml'

File: bimur/bimur_description/urdf/ur5.xacro (robot description, xacro)
@@ -25,5 +25,4 @@
    <xacro:arg name="safety_k_position" default="20"/>
   <xacro:ur5_robot
-    prefix=""
     joint_limits_parameters_file="$(arg joint_limit_params)"
     kinematics_parameters_file="$(arg kinematics_params)"
@@ -35,7 +34,6 @@
     safety_k_position="$(arg safety_k_position)"/>
   <!-- robotiq 85 -->
-  <xacro:include filename="$(find robotiq_85_description)/urdf/robotiq_85_gripper.urdf.xacro" />
+  <xacro:include filename="$(find robotiq_85_description)/urdf/robotiq_85_gripper.urdf.xacro"/>
   <link name="world"/>
-  <link name="ee_link" />
   <link name="frame">
     <inertial>
@@ -84,32 +82,38 @@
   </link>
   <joint name="frame_to_world" type="fixed">
+    <parent link="world"/>
+    <child link="frame"/>
+    <origin xyz="0.0 0.0 0.0" rpy="0.0 0.0 0.0" />
+  </joint>
+  <joint name="wall_to_world" type="fixed">
       <parent link="world"/>
-      <child link="frame"/>
-      <origin xyz="0.0 0.0 0.0" rpy="0.0 0.0 0.0" />
-    </joint>
-    <joint name="wall_to_world" type="fixed">
-        <parent link="world"/>
-        <child link="wall"/>
-        <origin xyz="0.5 1.02 1" rpy="1.57 0 0"/>
-    </joint>
-    <!-- right arm -->
-    <joint name="ur5_to_frame" type="fixed">
-      <parent link="frame"/>
-      <child link = "base_link"/>
-      <origin xyz="0.265 0.635 1.275" rpy="-0.785 3.14 1.57"/>
-    </joint>
-    <!-- astra camera -->
-    <link name="camera_mount"/>
-    <joint name="camera_to_frame" type="fixed">
-      <parent link="frame"/>
-      <child link = "camera_mount"/>
-      <origin xyz="0.54 0.54 1.45" rpy="0 1.30 -1.57"/>
-    </joint>
-    <!-- Right robotiq 85 -->
-    <xacro:robotiq_85_gripper prefix="" parent="ee_link" >
-      <origin xyz="0 0 0" rpy="0 0 0"/>
-    </xacro:robotiq_85_gripper>
-    <!-- Astra camera -->
-    <xacro:include filename="$(find bimur_description)/urdf/camera/astra.xacro"/>
-    <xacro:sensor_astra name="astra" parent="camera_mount" cam_px="0.01" cam_pz="${0.052}" meshes="package://bimur_description/meshes/rgbd" />
+      <child link="wall"/>
+      <origin xyz="0.5 1.02 1" rpy="1.57 0 0"/>
+  </joint>
+  <!-- right arm -->
+  <joint name="ur5_to_frame" type="fixed">
+    <parent link="frame"/>
+    <child link = "base_link"/>
+    <origin xyz="0.265 0.635 1.275" rpy="-0.785 3.14 1.57"/>
+  </joint>
+  <!-- astra camera -->
+  <link name="camera_mount"/>
+  <joint name="camera_to_frame" type="fixed">
+    <parent link="frame"/>
+    <child link = "camera_mount"/>
+    <origin xyz="0.54 0.54 1.45" rpy="0 1.30 -1.57"/>
+  </joint>
+  <link name="ee_link"/>
+  <joint name="link_to_ee" type="fixed">
+    <parent link="flange"/>
+    <child link = "ee_link"/>
+    <!-- <origin xyz="0.54 0.54 1.45" rpy="0 1.30 -1.57"/> -->
+  </joint>
+  <!-- Right robotiq 85 -->
+  <xacro:robotiq_85_gripper prefix="" parent="ee_link">
+    <origin xyz="0 0 0" rpy="0 0 0"/>
+  </xacro:robotiq_85_gripper>
+  <!-- Astra camera -->
+  <xacro:include filename="$(find bimur_description)/urdf/camera/astra.xacro"/>
+  <xacro:sensor_astra name="astra" parent="camera_mount" cam_px="0.01" cam_pz="${0.052}" meshes="package://bimur_description/meshes/rgbd" />
 </robot>

File: bimur/robotiq_85_gripper/robotiq_85_description/urdf/robotiq_85_gripper.urdf.xacro (robot description, xacro)
@@ -2,5 +2,7 @@
 <robot name="robotiq_85_gripper" xmlns:xacro="http://wiki.ros.org/xacro">
     <xacro:include filename="$(find robotiq_85_description)/urdf/robotiq_85_gripper.transmission.xacro" />
+    <!-- <link name="ee_link" /> -->
     <xacro:macro name="robotiq_85_gripper" params="prefix parent *origin">
+    <!-- <xacro:macro name="robotiq_85_gripper" params="prefix *origin"> -->
         <joint name="${prefix}gripper_base_joint" type="fixed">
             <parent link="${parent}"/>
